File: wiseboard.brd (EAGLE design)
At the start: 80 x 55 mm, 102 parts, among them IC1 MCP73871-2CCI/ML-ND, IC2 LM358MX, Q1 IRLML6402TRPBF, Q2 IRLML6402TRPBF, U1 LT1945EMSPBF, X1 1528-1438-ND

Commit message: CREATED BRANCH FOR TPS ALTERNATIVE POWER SOULTION
Connections:
- new net N$38: R36.1, R37.2
Changed lines of the file:
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@@
 <contactref element="U$20" pad="34"/>
+</signal>
+<signal name="N$38">
+<contactref element="R37" pad="2"/>
+<contactref element="R36" pad="1"/>
+<wire x1="-19.18" y1="-46.99" x2="-16.38" y2="-53.848" width="0" layer="19" extent="1-1"/>
 </signal>
 </signals>
