File: rev2/buttonboard.brd (EAGLE design)
At the start: 27.4 x 27.4 mm, 12 parts

Commit message: Add edge connectors to lbr, Prelim PCB layout, Consolidation, Fix mistakes
Parts:
- R6: value 33k -> 39k
Changed lines of the file:
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@@
 <attribute name="NAME" x="5.08" y="4.445" size="1.27" layer="25"/>
 </element>
-<element name="R6" library="resistor" library_urn="urn:adsk.eagle:library:348" package="R0805" value="33k" x="5.715" y="5.08" smashed="yes" rot="R180">
+<element name="R6" library="resistor" library_urn="urn:adsk.eagle:library:348" package="R0805" value="39k" x="5.715" y="5.08" smashed="yes" rot="R180">
 <attribute name="NAME" x="6.985" y="7.62" size="1.27" layer="25" rot="R180"/>
 </element>
