File: rev2/wiseboard.sch (EAGLE design)
At the start: 58 parts, among them IC1 LT1945, IC2 LM358, IC3 L79L15, IC4 L78L15, IC5 W25Q, IC8 IC6, IC9 BQ24210DQCT, J1 BAT_CON, J2 SOL_CON, J3 PROG_HEADER, J4 BUT_CON, Q1 IRLM, SW1 SPST_TACT-KMR2, SW2 SPST_TACT-KMR2, U3 ESP-WROOM-03

Commit message: Add test points make to do messages
Connections:
- removed net N$7: U3.IO0
- net +3V3: no longer U3.EN
- net GPIO0: now also U3.IO0
- net RESET: now also U3.EN
Changed lines of the file:
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@@
 <instance part="GND22" gate="1" x="91.44" y="-53.34" rot="R270"/>
 <instance part="R2" gate="G$1" x="-365.76" y="-33.02" rot="R270"/>
-<instance part="+3V3" gate="G$1" x="93.98" y="12.7" rot="R90"/>
+<instance part="+3V3" gate="G$1" x="86.36" y="15.24" rot="R90"/>
 <instance part="R1" gate="G$1" x="236.22" y="10.16" rot="R90"/>
 <instance part="R15" gate="G$1" x="236.22" y="0" rot="R90"/>
@@
 <junction x="0" y="60.96"/>
 </segment>
+<segment>
+<pinref part="U3" gate="G$1" pin="IO0"/>
+<wire x1="139.7" y1="7.62" x2="147.32" y2="7.62" width="0.1524" layer="91"/>
+<label x="144.78" y="7.62" size="1.778" layer="95"/>
+</segment>
 </net>
 <net name="RESET" class="0">
@@
 <pinref part="SW2" gate="G$1" pin="S1"/>
 <junction x="20.32" y="60.96"/>
+</segment>
+<segment>
+<pinref part="U3" gate="G$1" pin="EN"/>
+<wire x1="104.14" y1="12.7" x2="93.98" y2="12.7" width="0.1524" layer="91"/>
+<label x="93.98" y="12.7" size="1.778" layer="95"/>
 </segment>
 </net>
@@
 </segment>
 <segment>
-<pinref part="U3" gate="G$1" pin="EN"/>
-<wire x1="104.14" y1="12.7" x2="101.6" y2="12.7" width="0.1524" layer="91"/>
 <pinref part="+3V3" gate="G$1" pin="+3V3"/>
 <pinref part="U3" gate="G$1" pin="3V3"/>
-<wire x1="101.6" y1="12.7" x2="96.52" y2="12.7" width="0.1524" layer="91"/>
-<wire x1="104.14" y1="15.24" x2="101.6" y2="15.24" width="0.1524" layer="91"/>
-<wire x1="101.6" y1="15.24" x2="101.6" y2="12.7" width="0.1524" layer="91"/>
-<junction x="101.6" y="12.7"/>
+<wire x1="104.14" y1="15.24" x2="88.9" y2="15.24" width="0.1524" layer="91"/>
 </segment>
 </net>
@@
 </segment>
 </net>
-<net name="N$7" class="0">
-<segment>
-<pinref part="U3" gate="G$1" pin="IO0"/>
-<wire x1="139.7" y1="7.62" x2="147.32" y2="7.62" width="0.1524" layer="91"/>
-<label x="144.78" y="7.62" size="1.778" layer="95"/>
-</segment>
-</net>
