File: rev3/wiseboard.sch (EAGLE design)
At the start: 58 parts, among them IC1 LT1945, IC2 LM358, IC3 L79L15, IC4 L78L15, IC5 W25Q, IC6 AP2112, IC7 ESP-WROOM-03, IC9 BQ24210DQCT, J1 BAT_CON, J2 SOL_CON, J3 PROG_HEADER, J4 BUT_CON, Q2 IRLML6402TRPBF, SW1 SPST_TACT-KMR2, SW2 SPST_TACT-KMR2

Commit message: Add test points make to do messages
Parts:
- added TP2, TP3, TP4, TP5, TP6: TPSTP20R, testpad:TPSTP20R
- added TP7: TPSTP20SQ, testpad:TPSTP20SQ
Connections:
- net +5V: now also TP6.PP
- net GND: now also TP7.PP
- net GPIO0: now also TP3.PP
- net RESET: now also TP2.PP
- net RXD: now also TP5.PP
- net TXD: now also TP4.PP
Other:
- note added: "Check to see if we really need that diode."
- note added: "Double check GPIO0 and RESET test points"
- note added: "renumber test points"
- moved on the sheet: IC5
Changed lines of the file:
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@@
 <layer number="99" name="SpiceOrder" color="7" fill="1" visible="no" active="no"/>
 <layer number="100" name="Muster" color="7" fill="1" visible="no" active="no"/>
-<layer number="101" name="Patch_Top" color="12" fill="4" visible="no" active="yes"/>
+<layer number="101" name="Patch_Top" color="12" fill="4" visible="yes" active="yes"/>
 <layer number="102" name="Vscore" color="7" fill="1" visible="no" active="yes"/>
 <layer number="103" name="fp3" color="7" fill="1" visible="no" active="yes"/>
@@
 <part name="IC6" library="WISE" deviceset="AP2112" device=""/>
 <part name="GND3" library="supply1" library_urn="urn:adsk.eagle:library:371" deviceset="GND" device=""/>
+<part name="TP2" library="testpad" library_urn="urn:adsk.eagle:library:385" deviceset="TPS" device="TP20R"/>
+<part name="TP3" library="testpad" library_urn="urn:adsk.eagle:library:385" deviceset="TPS" device="TP20R"/>
+<part name="TP4" library="testpad" library_urn="urn:adsk.eagle:library:385" deviceset="TPS" device="TP20R"/>
+<part name="TP5" library="testpad" library_urn="urn:adsk.eagle:library:385" deviceset="TPS" device="TP20R"/>
+<part name="TP6" library="testpad" library_urn="urn:adsk.eagle:library:385" deviceset="TPS" device="TP20R"/>
+<part name="TP7" library="testpad" library_urn="urn:adsk.eagle:library:385" deviceset="TPS" device="TP20SQ"/>
 </parts>
 <sheets>
@@
 <wire x1="137.16" y1="111.76" x2="40.64" y2="111.76" width="0.1524" layer="94" style="shortdash"/>
 <text x="63.5" y="114.3" size="3.81" layer="94">Flash Memory Chip</text>
+<text x="228.6" y="101.6" size="1.778" layer="101">Check to see if we really need that diode.</text>
+<text x="228.6" y="99.06" size="1.778" layer="101">Double check GPIO0 and RESET test points</text>
+<text x="228.6" y="96.52" size="1.778" layer="101">renumber test points</text>
 </plain>
 <instances>
@@
 <instance part="R10" gate="G$1" x="220.98" y="-132.08" rot="R90"/>
 <instance part="GND15" gate="1" x="236.22" y="-139.7"/>
-<instance part="IC5" gate="G$1" x="86.36" y="76.2"/>
+<instance part="IC5" gate="G$1" x="88.9" y="76.2"/>
 <instance part="GND20" gate="1" x="60.96" y="68.58" rot="R270"/>
 <instance part="+3V13" gate="G$1" x="116.84" y="83.82" rot="R270"/>
@@
 <instance part="IC6" gate="U$2" x="-58.42" y="66.04"/>
 <instance part="GND3" gate="1" x="157.48" y="-114.3" rot="R270"/>
+<instance part="TP2" gate="G$1" x="264.16" y="55.88" rot="R270"/>
+<instance part="TP3" gate="G$1" x="264.16" y="60.96" rot="R270"/>
+<instance part="TP4" gate="G$1" x="264.16" y="66.04" rot="R270"/>
+<instance part="TP5" gate="G$1" x="264.16" y="71.12" rot="R270"/>
+<instance part="TP6" gate="G$1" x="264.16" y="76.2" rot="R270"/>
+<instance part="TP7" gate="G$1" x="264.16" y="81.28" rot="R270"/>
 </instances>
 <busses>
@@
 <segment>
 <pinref part="IC5" gate="G$1" pin="GND"/>
-<wire x1="68.58" y1="68.58" x2="63.5" y2="68.58" width="0.1524" layer="91"/>
+<wire x1="71.12" y1="68.58" x2="63.5" y2="68.58" width="0.1524" layer="91"/>
 <pinref part="GND20" gate="1" pin="GND"/>
 </segment>
@@
 <pinref part="GND3" gate="1" pin="GND"/>
 <wire x1="160.02" y1="-114.3" x2="162.56" y2="-114.3" width="0.1524" layer="91"/>
+</segment>
+<segment>
+<pinref part="TP7" gate="G$1" pin="PP"/>
+<wire x1="261.62" y1="81.28" x2="254" y2="81.28" width="0.1524" layer="91"/>
+<label x="254" y="81.28" size="1.778" layer="95"/>
 </segment>
 </net>
@@
 <label x="144.78" y="15.24" size="1.778" layer="95"/>
 </segment>
+<segment>
+<pinref part="TP4" gate="G$1" pin="PP"/>
+<wire x1="261.62" y1="66.04" x2="254" y2="66.04" width="0.1524" layer="91"/>
+<label x="254" y="66.04" size="1.778" layer="95"/>
+</segment>
 </net>
 <net name="GPIO0" class="0">
@@
 <label x="144.78" y="7.62" size="1.778" layer="95"/>
 </segment>
+<segment>
+<pinref part="TP3" gate="G$1" pin="PP"/>
+<wire x1="261.62" y1="60.96" x2="254" y2="60.96" width="0.1524" layer="91"/>
+<label x="254" y="60.96" size="1.778" layer="95"/>
+</segment>
 </net>
 <net name="RESET" class="0">
@@
 <label x="93.98" y="12.7" size="1.778" layer="95"/>
 </segment>
+<segment>
+<pinref part="TP2" gate="G$1" pin="PP"/>
+<wire x1="261.62" y1="55.88" x2="254" y2="55.88" width="0.1524" layer="91"/>
+<label x="254" y="55.88" size="1.778" layer="95"/>
+</segment>
 </net>
 <net name="+3V3" class="0">
@@
 <segment>
 <pinref part="IC5" gate="G$1" pin="VCC"/>
-<wire x1="104.14" y1="83.82" x2="114.3" y2="83.82" width="0.1524" layer="91"/>
+<wire x1="106.68" y1="83.82" x2="114.3" y2="83.82" width="0.1524" layer="91"/>
 <pinref part="+3V13" gate="G$1" pin="+3V3"/>
 </segment>
 <segment>
 <pinref part="IC5" gate="G$1" pin="WP"/>
-<wire x1="68.58" y1="73.66" x2="53.34" y2="73.66" width="0.1524" layer="91"/>
+<wire x1="71.12" y1="73.66" x2="53.34" y2="73.66" width="0.1524" layer="91"/>
 <pinref part="+3V14" gate="G$1" pin="+3V3"/>
 </segment>
@@
 <wire x1="139.7" y1="12.7" x2="147.32" y2="12.7" width="0.1524" layer="91"/>
 <label x="144.78" y="12.7" size="1.778" layer="95"/>
+</segment>
+<segment>
+<pinref part="TP5" gate="G$1" pin="PP"/>
+<wire x1="261.62" y1="71.12" x2="254" y2="71.12" width="0.1524" layer="91"/>
+<label x="254" y="71.12" size="1.778" layer="95"/>
 </segment>
 </net>
@@
 <segment>
 <pinref part="IC5" gate="G$1" pin="DI"/>
-<wire x1="104.14" y1="68.58" x2="114.3" y2="68.58" width="0.1524" layer="91"/>
+<wire x1="106.68" y1="68.58" x2="114.3" y2="68.58" width="0.1524" layer="91"/>
 <label x="111.76" y="68.58" size="1.778" layer="95"/>
 </segment>
@@
 <segment>
 <pinref part="IC5" gate="G$1" pin="CLK"/>
-<wire x1="104.14" y1="73.66" x2="116.84" y2="73.66" width="0.1524" layer="91"/>
+<wire x1="106.68" y1="73.66" x2="116.84" y2="73.66" width="0.1524" layer="91"/>
 <label x="111.76" y="73.66" size="1.778" layer="95"/>
 </segment>
@@
 <segment>
 <pinref part="IC5" gate="G$1" pin="DO"/>
-<wire x1="68.58" y1="78.74" x2="58.42" y2="78.74" width="0.1524" layer="91"/>
+<wire x1="71.12" y1="78.74" x2="58.42" y2="78.74" width="0.1524" layer="91"/>
 <label x="58.42" y="78.74" size="1.778" layer="95"/>
 </segment>
@@
 <pinref part="IC6" gate="U$2" pin="VIN"/>
 </segment>
+<segment>
+<pinref part="TP6" gate="G$1" pin="PP"/>
+<wire x1="261.62" y1="76.2" x2="254" y2="76.2" width="0.1524" layer="91"/>
+<label x="254" y="76.2" size="1.778" layer="95"/>
+</segment>
 </net>
 <net name="N$6" class="0">
@@
 <segment>
 <pinref part="IC5" gate="G$1" pin="CS"/>
-<wire x1="68.58" y1="83.82" x2="60.96" y2="83.82" width="0.1524" layer="91"/>
-</segment>
-</net>
+<wire x1="71.12" y1="83.82" x2="60.96" y2="83.82" width="0.1524" layer="91"/>
+</segment>
+</net>

Commit message: Start new pcb
Parts:
- removed D6: SS24, WISE:SS24
- added 3V3: TPSTP20R, testpad:TPSTP20R
- C3: value 1uF -> 0.1uF
- D1: value MBR120VLSFT1G -> MBR120; device microbuilder:DIODESOD-123 -> adafruit:DIODESOD-123
- D2: value MBR120 -> 1n4148
- D3: value 1n4148 -> SS24; device adafruit:DIODESOD-123 -> WISE:SS24
- renumbered TP2 to RST, TP3 to IO0, TP4 to TXD, TP5 to RXD, TP6 to 5V, TP7 to GND
Connections:
- removed net N$3: C8.2, D1.C, IC9.VBUS
- removed net VOUT: IC6.VOUT
- net +22V: now also D5.C; no longer D6.C
- net +3V3: now also 3V3.PP, IC6.VOUT
- net +5V: now also D1.C; no longer D2.C
- net -20V: now also D3.A; no longer D5.A
- net GND: now also IC4.GND; no longer IC4.GND@2, IC4.GND@6, IC4.GND@7
- net N$5: now also D5.A; no longer D6.A
- net N$6: now also D3.C; no longer D5.C
- net PANEL: now also C8.2, IC9.VBUS; no longer D1.A
- net RXD: now also D2.A; no longer D3.A
- net RXD_5V: now also D2.C; no longer D3.C
- net VBAT: now also D1.A; no longer D2.A
Other:
- note added: "some caps should be rated for >25v"
- moved on the sheet: D1, D2, D5, IC4

Commit message: finish layout of PCB
Parts:
- added +15V, +22V, -15V, -20V: TPSTP20R, testpad:TPSTP20R
- added GND17: TPSTP20SQ, testpad:TPSTP20SQ
Connections:
- net +15V: now also +15V.PP
- net +22V: now also +22V.PP
- net -15V: now also -15V.PP
- net -20V: now also -20V.PP
- net GND: now also GND17.PP
Changed lines of the file:
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@@
 <part name="+3V7" library="supply1" library_urn="urn:adsk.eagle:library:371" deviceset="+3V3" device=""/>
 <part name="+3V1" library="supply1" library_urn="urn:adsk.eagle:library:371" deviceset="+3V3" device=""/>
+<part name="-15V" library="testpad" library_urn="urn:adsk.eagle:library:385" deviceset="TPS" device="TP20R"/>
+<part name="+15V" library="testpad" library_urn="urn:adsk.eagle:library:385" deviceset="TPS" device="TP20R"/>
+<part name="-20V" library="testpad" library_urn="urn:adsk.eagle:library:385" deviceset="TPS" device="TP20R"/>
+<part name="+22V" library="testpad" library_urn="urn:adsk.eagle:library:385" deviceset="TPS" device="TP20R"/>
+<part name="GND10" library="supply1" library_urn="urn:adsk.eagle:library:371" deviceset="GND" device=""/>
+<part name="GND17" library="testpad" library_urn="urn:adsk.eagle:library:385" deviceset="TPS" device="TP20SQ"/>
 </parts>
 <sheets>
@@
 <instance part="+3V7" gate="G$1" x="-50.8" y="83.82" rot="R270"/>
 <instance part="+3V1" gate="G$1" x="-33.02" y="71.12" rot="R270"/>
+<instance part="-15V" gate="G$1" x="-93.98" y="15.24"/>
+<instance part="+15V" gate="G$1" x="-93.98" y="-55.88"/>
+<instance part="-20V" gate="G$1" x="-175.26" y="10.16"/>
+<instance part="+22V" gate="G$1" x="-170.18" y="-58.42"/>
+<instance part="GND10" gate="1" x="-63.5" y="7.62"/>
+<instance part="GND17" gate="G$1" x="-63.5" y="12.7"/>
 </instances>
 <busses>
@@
 <pinref part="GND11" gate="1" pin="GND"/>
 <junction x="-162.56" y="-73.66"/>
+</segment>
+<segment>
+<pinref part="GND10" gate="1" pin="GND"/>
+<pinref part="GND17" gate="G$1" pin="PP"/>
 </segment>
 </net>
@@
 <wire x1="-127" y1="-66.04" x2="-119.38" y2="-66.04" width="0.1524" layer="91"/>
 <wire x1="-119.38" y1="-66.04" x2="-104.14" y2="-66.04" width="0.1524" layer="91"/>
-<wire x1="-104.14" y1="-66.04" x2="-81.28" y2="-66.04" width="0.1524" layer="91"/>
+<wire x1="-104.14" y1="-66.04" x2="-93.98" y2="-66.04" width="0.1524" layer="91"/>
 <pinref part="C6" gate="G$1" pin="1"/>
+<wire x1="-93.98" y1="-66.04" x2="-81.28" y2="-66.04" width="0.1524" layer="91"/>
 <wire x1="-119.38" y1="-81.28" x2="-119.38" y2="-66.04" width="0.1524" layer="91"/>
 <junction x="-119.38" y="-66.04"/>
@@
 <junction x="-104.14" y="-66.04"/>
 <label x="-86.36" y="-66.04" size="1.778" layer="95"/>
+<pinref part="+15V" gate="G$1" pin="PP"/>
+<wire x1="-93.98" y1="-58.42" x2="-93.98" y2="-66.04" width="0.1524" layer="91"/>
+<junction x="-93.98" y="-66.04"/>
 </segment>
 <segment>
@@
 <junction x="-114.3" y="2.54"/>
 <wire x1="-101.6" y1="2.54" x2="-101.6" y2="-5.08" width="0.1524" layer="91"/>
-<wire x1="-101.6" y1="2.54" x2="-81.28" y2="2.54" width="0.1524" layer="91"/>
+<wire x1="-101.6" y1="2.54" x2="-93.98" y2="2.54" width="0.1524" layer="91"/>
 <junction x="-101.6" y="2.54"/>
 <label x="-86.36" y="2.54" size="1.778" layer="95"/>
+<pinref part="-15V" gate="G$1" pin="PP"/>
+<wire x1="-93.98" y1="2.54" x2="-81.28" y2="2.54" width="0.1524" layer="91"/>
+<wire x1="-93.98" y1="12.7" x2="-93.98" y2="2.54" width="0.1524" layer="91"/>
+<junction x="-93.98" y="2.54"/>
 </segment>
 <segment>
@@
 <junction x="-190.5" y="-5.08"/>
 <junction x="-177.8" y="-5.08"/>
-<wire x1="-177.8" y1="-5.08" x2="-165.1" y2="-5.08" width="0.1524" layer="91"/>
+<wire x1="-177.8" y1="-5.08" x2="-175.26" y2="-5.08" width="0.1524" layer="91"/>
+<wire x1="-175.26" y1="-5.08" x2="-165.1" y2="-5.08" width="0.1524" layer="91"/>
 <wire x1="-165.1" y1="-5.08" x2="-160.02" y2="-5.08" width="0.1524" layer="91"/>
 <wire x1="-165.1" y1="-5.08" x2="-165.1" y2="-12.7" width="0.1524" layer="91"/>
@@
 <wire x1="-119.38" y1="-12.7" x2="-129.54" y2="-12.7" width="0.1524" layer="91"/>
 <junction x="-129.54" y="-12.7"/>
-<label x="-172.72" y="-5.08" size="1.778" layer="95"/>
+<label x="-167.64" y="-5.08" size="1.778" layer="95"/>
+<pinref part="-20V" gate="G$1" pin="PP"/>
+<wire x1="-175.26" y1="7.62" x2="-175.26" y2="-5.08" width="0.1524" layer="91"/>
+<junction x="-175.26" y="-5.08"/>
 </segment>
 <segment>
@@
 <junction x="-177.8" y="-66.04"/>
 <pinref part="IC4" gate="G$1" pin="VIN"/>
-<wire x1="-177.8" y1="-66.04" x2="-157.48" y2="-66.04" width="0.1524" layer="91"/>
-<label x="-170.18" y="-66.04" size="1.778" layer="95"/>
-</segment>
-<segment>
+<wire x1="-177.8" y1="-66.04" x2="-170.18" y2="-66.04" width="0.1524" layer="91"/>
+<label x="-165.1" y="-66.04" size="1.778" layer="95"/>
+<pinref part="+22V" gate="G$1" pin="PP"/>
+<wire x1="-170.18" y1="-66.04" x2="-157.48" y2="-66.04" width="0.1524" layer="91"/>
+<wire x1="-170.18" y1="-60.96" x2="-170.18" y2="-66.04" width="0.1524" layer="91"/>
+<junction x="-170.18" y="-66.04"/>
+</segment>
+<segment>

Commit message: Fix REST GPIO0 Intersection
Parts:
- added 5V1, IO1, RST1, RXD1, TXD1: TPSTP20R, testpad:TPSTP20R
- added GND23: TPSTP20SQ, testpad:TPSTP20SQ
- C1, C6: value 1uF -> 1uF > 15V
- C10, C8: value 10uF -> 1uF
- C2: value 1uF -> 4.7uF
- C3: value 0.1uF -> 1uF
- C4: value 10uF -> 100pF
- C5: value 10uF -> 4.7pF > 22V
- R3: value 470k -> 560k > 20V
- R4: value 39k -> 39k > 20V
Connections:
- removed net N$48: IC7.IO34
- net +5V: now also 5V1.PP
- net GMODE: now also IC7.IO34
- net GND: now also GND23.PP
- net GPIO0: now also IO1.PP
- net RESET: now also RST1.PP
- net RXD: now also RXD1.PP
- net TXD: now also TXD1.PP
Other:
- note added: "GMODe is on pin 34"
- moved on the sheet: C5
